Commit message: Modified the urdf file

File: urdf/robot.urdf (robot description, URDF)
Before this commit: robot SBR, 1 links, 0 joints
Links:
- added link base_footprint
- added link left_wheel, mass 1.0; collision mesh filename=file:///$(find gazebo_visualization)/meshes/left_wheel.STL; visual mesh filename=file:///$(find gazebo_visualization)/meshes/left_wheel.STL
- added link right_wheel, mass 1.0; collision mesh filename=file:///$(find gazebo_visualization)/meshes/right_wheel.STL; visual mesh filename=file:///$(find gazebo_visualization)/meshes/right_wheel.STL
Joints:
- added joint base_joint: type fixed, parent base_link, child base_footprint, origin xyz=0 0 -0.350 rpy=0 0 0
- added joint base_left_wheel_joint: type continuous, parent base_link, child left_wheel, origin xyz=0 0 0 rpy=0 0 0, axis 0 1 0
- added joint base_right_wheel_joint: type continuous, parent base_link, child right_wheel, origin xyz=0 0 0 rpy=0 0 0, axis 0 1 0
